File: Distributor/hw/Grabber.kicad_sch (KiCad schematic)
At the start: 24 parts, among them J7 Conn_01x04, J8 Conn_01x06_MountingPin, J9 Conn_02x09_Odd_Even, U7 STM32F407VETx, U8 MLX90640ESF-BAB-000-TU

Commit message: I hate layout
Parts:
- removed C21: 100n, Capacitor_SMD:C_0603_1608Metric, symbol Device:C
- renumbered C22 to C21, C23 to C22, C24 to C23, C25 to C24
Changed lines of the file:
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@@
   (junction (at 59.69 139.065) (diameter 0) (color 0 0 0 0)
   )
-  (junction (at 223.52 32.385) (diameter 0) (color 0 0 0 0)
-  )
   (junction (at 189.23 24.765) (diameter 0) (color 0 0 0 0)
   )
@@
   )
   (junction (at 142.875 24.765) (diameter 0) (color 0 0 0 0)
-  )
-  (junction (at 223.52 24.765) (diameter 0) (color 0 0 0 0)
   )
   (junction (at 177.8 32.385) (diameter 0) (color 0 0 0 0)
@@
     (stroke (width 0) (type default))
   )
-  (wire (pts (xy 223.52 24.765) (xy 234.95 24.765))
-    (stroke (width 0) (type default))
-  )
   (wire (pts (xy 34.29 76.2) (xy 39.37 76.2))
     (stroke (width 0) (type default))
@@
   )
   (wire (pts (xy 55.245 115.57) (xy 51.435 115.57))
-    (stroke (width 0) (type default))
-  )
-  (wire (pts (xy 223.52 32.385) (xy 234.95 32.385))
     (stroke (width 0) (type default))
   )
@@
     (effects (font (size 1.27 1.27) italic) (justify left bottom))
   )
-  (text "Decp. VREF/VDDA-VSSA" (at 226.06 35.56 0)
+  (text "Decp. VREF/VDDA-VSSA" (at 214.63 35.56 0)
     (effects (font (size 1.27 1.27) italic) (justify left bottom))
   )
@@
   (symbol (lib_id "Device:C") (at 71.12 142.875 0) (unit 1)
     (in_bom yes) (on_board yes) (dnp no)
-    (property "Reference" "C25" (at 74.295 141.605 0)
+    (property "Reference" "C24" (at 74.295 141.605 0)
       (effects (font (size 1.27 1.27)) (justify left))
     )
@@
       (project "Distributor"
         (path "/3f67d80a-1b5b-4b57-a63e-46eb7de4787a/d071538b-874a-4835-97d2-570c76260972"
-          (reference "C25") (unit 1)
+          (reference "C24") (unit 1)
         )
       )
@@
     )
   )
-  (symbol (lib_id "Device:C") (at 234.95 28.575 0) (unit 1)
-    (in_bom yes) (on_board yes) (dnp no)
-    (property "Reference" "C21" (at 238.125 27.305 0)
-      (effects (font (size 1.27 1.27)) (justify left))
-    )
-    (property "Value" "100n" (at 238.125 29.845 0)
-      (effects (font (size 1.27 1.27)) (justify left))
-    )
-    (property "Footprint" "Capacitor_SMD:C_0603_1608Metric" (at 235.9152 32.385 0)
-      (effects (font (size 1.27 1.27)) hide)
-    )
-    (property "Datasheet" "~" (at 234.95 28.575 0)
-      (effects (font (size 1.27 1.27)) hide)
-    )
-    (pin "1")
-    (pin "2")
-    (instances
-      (project "Distributor"
-        (path "/3f67d80a-1b5b-4b57-a63e-46eb7de4787a/d071538b-874a-4835-97d2-570c76260972"
-          (reference "C21") (unit 1)
-        )
-      )
-    )
-  )
   (symbol (lib_id "Device:C") (at 189.23 28.575 0) (unit 1)
     (in_bom yes) (on_board yes) (dnp no)
@@
   (symbol (lib_id "Device:C") (at 59.69 142.875 0) (unit 1)
     (in_bom yes) (on_board yes) (dnp no)
-    (property "Reference" "C24" (at 62.865 141.605 0)
+    (property "Reference" "C23" (at 62.865 141.605 0)
       (effects (font (size 1.27 1.27)) (justify left))
     )
@@
       (project "Distributor"
         (path "/3f67d80a-1b5b-4b57-a63e-46eb7de4787a/d071538b-874a-4835-97d2-570c76260972"
-          (reference "C24") (unit 1)
+          (reference "C23") (unit 1)
         )
       )
@@
   (symbol (lib_id "Device:C") (at 104.14 153.67 0) (mirror y) (unit 1)
     (in_bom yes) (on_board yes) (dnp no)
-    (property "Reference" "C23" (at 100.965 152.4 0)
+    (property "Reference" "C22" (at 100.965 152.4 0)
       (effects (font (size 1.27 1.27)) (justify left))
     )
@@
       (project "Distributor"
         (path "/3f67d80a-1b5b-4b57-a63e-46eb7de4787a/d071538b-874a-4835-97d2-570c76260972"
-          (reference "C23") (unit 1)
+          (reference "C22") (unit 1)
         )
       )
@@
   (symbol (lib_id "Device:C") (at 93.345 151.13 0) (mirror y) (unit 1)
     (in_bom yes) (on_board yes) (dnp no)
-    (property "Reference" "C22" (at 90.17 149.86 0)
+    (property "Reference" "C21" (at 90.17 149.86 0)
       (effects (font (size 1.27 1.27)) (justify left))
     )
@@
       (project "Distributor"
         (path "/3f67d80a-1b5b-4b57-a63e-46eb7de4787a/d071538b-874a-4835-97d2-570c76260972"
-          (reference "C22") (unit 1)
-        )
-      )
+          (reference "C21") (unit 1)
+        )
+      )
