File: Distributor/hw/Grabber.kicad_sch (KiCad schematic)
At the start: 23 parts, among them J7 Conn_01x04, J8 Conn_01x06_MountingPin, J9 Conn_02x09_Odd_Even, U7 STM32F407VETx, U8 MLX90640ESF-BAB-000-TU

Commit message: Fix wrong value of capacitors on VCAP pins
Parts:
- C21, C22: value 100n -> 2.2u
Changed lines of the file:
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@@
       (effects (font (size 1.27 1.27)) (justify left))
     )
-    (property "Value" "100n" (at 100.965 154.94 0)
+    (property "Value" "2.2u" (at 100.965 154.94 0)
       (effects (font (size 1.27 1.27)) (justify left))
     )
@@
       (effects (font (size 1.27 1.27)) (justify left))
     )
-    (property "Value" "100n" (at 90.17 152.4 0)
+    (property "Value" "2.2u" (at 90.17 152.4 0)
       (effects (font (size 1.27 1.27)) (justify left))
     )

Commit message: Update EDA document with actual values in assembly
Parts:
- D7: value White -> Green
- D8: value White -> Yellow
- R8: value 4.7k TBD -> 10k
- R9: value 4.7k TBD -> 7.5k
Changed lines of the file:
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@@
       (effects (font (size 1.27 1.27)))
     )
-    (property "Value" "4.7k TBD" (at 53.975 83.185 90)
+    (property "Value" "7.5k" (at 53.975 83.185 90)
       (effects (font (size 1.27 1.27)))
     )
@@
       (effects (font (size 1.27 1.27)))
     )
-    (property "Value" "White" (at 44.45 72.39 0)
+    (property "Value" "Green" (at 44.45 72.39 0)
       (effects (font (size 1.27 1.27)))
     )
@@
       (effects (font (size 1.27 1.27)))
     )
-    (property "Value" "4.7k TBD" (at 53.975 73.025 90)
+    (property "Value" "10k" (at 53.975 73.025 90)
       (effects (font (size 1.27 1.27)))
     )
@@
       (effects (font (size 1.27 1.27)))
     )
-    (property "Value" "White" (at 44.45 82.55 0)
-      (effects (font (size 1.27 1.27)))
-    )
+    (property "Value" "Yellow" (at 44.45 82.55 0)
+      (effects (font (size 1.27 1.27)))
+    )
