File: Distributor/hw/Distributor.kicad_pcb (KiCad board)
At the start: 2 copper layers, 77 parts, among them J1 Conn_01x04, J100 Conn_01x03, J101 Conn_01x03, J102 Conn_01x03, J103 Conn_01x03, J104 Conn_01x03, J105 Conn_01x03, J106 Conn_01x03, J107 Conn_01x03, J108 Conn_01x03, J109 Conn_01x03, J110 Conn_01x03, J111 Conn_01x03, J112 Conn_01x03, J113 Conn_01x03, J114 Conn_01x03, J115 Conn_01x03, J116 Conn_01x03, J117 Conn_01x03, J118 Conn_01x03, J119 Conn_01x03, J120 Conn_01x03, J121 Conn_01x03, J122 Conn_01x03, J123 Conn_01x03, J124 Conn_01x03, J125 Conn_01x03, J126 Conn_01x03, J127 Conn_01x03, J128 Conn_01x03, J129 Conn_01x03, J130 Conn_01x03, J131 Conn_01x03, J2 Conn_01x06_MountingPin, J3 Conn_01x02, J4 Conn_01x02, J5 Conn_01x02, J6 Conn_01x02, J7 Conn_01x04, J8 Conn_01x06_MountingPin, J9 Conn_02x09_Odd_Even, U1 SPX3819M5-L-3-3, U2 STM32G030C8Tx, U3 SN74AHCT245PWR, U4 SN74AHCT245PWR, U5 SN74AHCT245PWR, U6 SN74AHCT245PWR, U7 STM32G070CBTx, U8 MLX90640ESF-BAB-000-TU

Commit message: Board layout
Parts:
- moved J6 125.5 mm to (16.5, 21.5)
- moved C9 120.7 mm to (143.5, 22.5)
- moved C12 111.1 mm to (23.5, 22.5), turned to -90 degrees
- moved J5 80.9 mm to (56.5, 21.5)
- moved D2 80.3 mm to (95.2, 50.2)
- moved D1 80.0 mm to (95.2, 48.8)
- moved D4 73.4 mm to (41.7, 36.1), turned to 90 degrees
- moved J8 71.5 mm to (45.5, 46.6), turned to 90 degrees
- moved U1 71.2 mm to (100.7, 47.8), turned to 180 degrees
- moved D3 70.9 mm to (40.2, 36.1), turned to 90 degrees
- moved C11 69.9 mm to (63.5, 22.5), turned to -90 degrees
- moved R6 68.6 mm to (40.2, 39.1), turned to -90 degrees
- moved R5 66.4 mm to (41.7, 39.1), turned to -90 degrees
- moved C5 66.2 mm to (156.7, 30.3)
- moved U3 66.2 mm to (161.0, 31.1)
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Connections:
- U1 pad 1: +5V-D -> +5V-A
- U1 pad 3: +5V-D -> +5V-A
- U2 pad 5: GND -> VDD
- U7 pad 5: GND -> VDD

Commit message: 🚧 Board routing
Parts:
- moved J2 15.2 mm to (55.2, 46.6)
- moved C2 3.42 mm to (97.8, 47.5), turned to -90 degrees
- moved U6 2.83 mm to (52.0, 33.1)
- moved C8 2.83 mm to (47.6, 32.3)
- moved D1 1.50 mm to (95.2, 50.2)
- moved D2 1.50 mm to (95.2, 48.8)
- moved C5 0.50 mm to (156.7, 30.8)
- moved C6 0.50 mm to (116.6, 30.8)
- moved U3 0.50 mm to (161.0, 31.6)
- moved U4 0.50 mm to (121.0, 31.6)
Routing:
- net LS0: track 0.00 -> 79.7 mm, vias 0 -> 2
- net LS1: track 0.00 -> 77.7 mm
- net LS2: track 0.00 -> 74.6 mm
- net LS3: track 0.00 -> 73.8 mm
- net LS4: track 0.00 -> 72.9 mm
- net LS5: track 0.00 -> 72.1 mm
- net LS6: track 0.00 -> 71.2 mm
- net LS7: track 0.00 -> 70.4 mm
- net LS31: track 0.00 -> 38.0 mm
- net LS30: track 0.00 -> 37.1 mm
- net LS29: track 0.00 -> 36.3 mm
- net LS28: track 0.00 -> 35.4 mm
- net LS8: track 0.00 -> 34.9 mm
- net LS27: track 0.00 -> 34.5 mm
- net LS26: track 0.00 -> 33.7 mm
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- added copper zone on B.Cu, net +5V-A
- added copper zone on F.Cu, net +5V-A
- added copper zone on B.Cu, net +5V-B
- added copper zone on F.Cu, net +5V-B
- added copper zone on B.Cu, net +5V-C
- added copper zone on F.Cu, net +5V-C
- added copper zone on B.Cu, net +5V-D
- added copper zone on F.Cu, net +5V-D
- added copper zone on B.Cu, net GND
- added copper zone on F.Cu, net GND
- added copper zone on F.Cu, net VDD

Commit message: Finish routing
Parts:
- moved D4 1.50 mm to (40.2, 36.1)
- moved D3 1.47 mm to (41.7, 36.1)
- moved R7 0.27 mm to (26.1, 45.9)
- moved R8 0.27 mm to (27.6, 45.9)
- moved J7 0.05 mm to (28.9, 50.4)
Connections:
- U7 pad 13: unconnected-(U7-PA2-Pad13) -> /Grabber/CAM_HREF
- U7 pad 14: /Grabber/CAM_RESET -> /Grabber/CAM_PWDN
- U7 pad 15: /Grabber/CAM_PWDN -> /Grabber/CAM_RESET
- U7 pad 16: /Grabber/CAM_VSYNC -> unconnected-(U7-PA5-Pad16)
- U7 pad 17: /Grabber/CAM_HREF -> unconnected-(U7-PA6-Pad17)
- U7 pad 18: /Grabber/CAM_PCLK -> unconnected-(U7-PA7-Pad18)
- U7 pad 27: unconnected-(U7-PB15-Pad27) -> /Grabber/CAM_PCLK
- U7 pad 29: unconnected-(U7-PA9/NC-Pad29) -> /Grabber/CAM_VSYNC
Routing:
- net VDD: track 15.6 -> 133.9 mm, vias 2 -> 6
- net +5V-A: track 24.7 -> 107.5 mm
- net /SPI_CK: track 0.00 -> 52.3 mm, vias 0 -> 2
- net /SPI_DI: track 0.00 -> 52.1 mm, vias 0 -> 2
- net /SPI_CS: track 0.00 -> 50.0 mm, vias 0 -> 2
- net /Grabber/CAM_HREF: track 0.00 -> 24.6 mm
- net /Grabber/SDA: track 0.00 -> 23.6 mm, vias 0 -> 2
- net GND: track 21.6 -> 45.0 mm, vias 14 -> 25
- net /Grabber/SCL: track 0.00 -> 22.5 mm
- net /SWCLK: track 0.00 -> 14.7 mm
- net /SWDIO: track 0.00 -> 12.8 mm
- net /Grabber/CAM_XCLK: track 0.00 -> 12.8 mm
- net /Grabber/CAM_VSYNC: track 0.00 -> 11.1 mm
- net /Grabber/CAM_D6: track 0.00 -> 8.72 mm
- net /Grabber/CAM_PCLK: track 0.00 -> 8.42 mm
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Other:
- board outline added: 155.1 x 39.1 mm
- board text added: "+"
- board text added: "+5V"
- board text added: "-"
- board text added: "A"
- board text added: "B"
- board text added: "C"
- board text added: "D"

Commit message: Revise distributor board; submit for fab
Parts:
- added D3: Green, LED_SMD:LED_0603_1608Metric, F.Cu at (148.4, 27.9)
- added D4: Green, LED_SMD:LED_0603_1608Metric, F.Cu at (108.5, 27.9)
- added D5: Green, LED_SMD:LED_0603_1608Metric, F.Cu at (68.5, 27.9)
- added D6: Green, LED_SMD:LED_0603_1608Metric, F.Cu at (28.4, 27.9)
- added G***: LOGO, LOGO, F.Cu at (166.9, 43.8)
- added G***: LOGO, LOGO, F.Cu at (167.2, 48.6)
- added G***: LOGO, LOGO, B.Cu at (46.8, 49.0)
- added R4: 6.8k TBD, Resistor_SMD:R_0603_1608Metric, F.Cu at (148.4, 29.4)
- added R5: 6.8k TBD, Resistor_SMD:R_0603_1608Metric, F.Cu at (108.5, 29.4)
- added R6: 6.8k TBD, Resistor_SMD:R_0603_1608Metric, F.Cu at (68.5, 29.4)
- added R7: 6.8k TBD, Resistor_SMD:R_0603_1608Metric, F.Cu at (28.4, 29.4)
- renumbered D3 to D7, D4 to D8, R6 to R10, R7 to R11, R8 to R12, R4 to R8, R5 to R9
Routing:
- net GND: track 45.0 -> 47.9 mm, vias 25 -> 29
- net Net-(D6-K): track 0.00 -> 1.52 mm
- net Net-(D5-K): track 0.00 -> 1.52 mm
- net Net-(D4-K): track 0.00 -> 1.52 mm
- net Net-(D3-K): track 0.00 -> 1.52 mm
- net +5V-C: track 21.0 -> 22.4 mm
- net +5V-B: track 21.5 -> 23.0 mm
- net +5V-D: track 33.0 -> 34.5 mm
- net +5V-A: track 107.5 -> 109.0 mm
Other:
- outline, holes or cut-outs redrawn
- board text added: "24-Soak"
- board text added: "Rev. 1"

Commit message: I hate layout
Parts:
- removed the R8 at (28.9, 48.8)
- added C15: 100n, Capacitor_SMD:C_0603_1608Metric, F.Cu at (-151.3, 39.1)
- added C16: 100n, Capacitor_SMD:C_0603_1608Metric, F.Cu at (-156.3, 33.0)
- added C17: 100n, Capacitor_SMD:C_0603_1608Metric, F.Cu at (-168.3, 33.7)
- added C18: 100n, Capacitor_SMD:C_0603_1608Metric, F.Cu at (-171.2, 48.3)
- added C19: 100n, Capacitor_SMD:C_0603_1608Metric, F.Cu at (-152.2, 50.3)
- added C20: 1u, Capacitor_SMD:C_0603_1608Metric, F.Cu at (-149.7, 39.1)
- added C21: 100n, Capacitor_SMD:C_0603_1608Metric, F.Cu at (-166.8, 32.2)
- added C22: 100n, Capacitor_SMD:C_0603_1608Metric, F.Cu at (-171.2, 46.8)
- U7: value STM32G070CBTx -> STM32F407VETx; footprint Package_QFP:LQFP-48_7x7mm_P0.5mm -> Package_QFP:LQFP-100_14x14mm_P0.5mm
- moved G*** 250.0 mm to (-203.2, 49.0)
- moved J9 205.9 mm to (-188.8, 49.9), turned to 180 degrees
- moved C12 205.5 mm to (-182.0, 22.5)
- moved J131 205.0 mm to (-175.0, 20.0)
- moved J7 201.7 mm to (-172.7, 50.2), turned to 0 degrees
- moved R11 200.5 mm to (-172.4, 31.8), turned to 180 degrees
- moved C23 199.0 mm to (-181.6, 41.8), turned to -67.5 degrees
- moved R10 199.0 mm to (-172.4, 33.2), turned to 180 degrees
- moved C24 198.2 mm to (-180.2, 41.2), turned to -67.5 degrees
- moved U8 196.1 mm to (-173.2, 36.7), turned to 180 degrees
- moved U7 195.3 mm to (-160.9, 42.5)
- moved G*** 193.1 mm to (360.0, 43.8)
- moved G*** 193.1 mm to (360.2, 48.6)
- moved C13 191.5 mm to (-149.8, 43.6), turned to -90 degrees
- moved C14 191.5 mm to (-151.3, 43.6), turned to -90 degrees
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- renumbered C15 to C23, C16 to C24, R11 to R10, R12 to R11, R9 to R8, R10 to R9
Connections:
- U2 pad 27: LS16 -> LS23
- U2 pad 28: LS17 -> LS22
- U2 pad 29: LS18 -> LS21
- U2 pad 30: LS19 -> LS20
- U2 pad 31: LS20 -> LS19
- U2 pad 32: LS21 -> LS18
- U2 pad 33: LS22 -> LS17
- U2 pad 34: LS23 -> LS16
- U7 pad 10: unconnected-(U7-NRST-Pad10) -> GND
- U7 pad 11: /Grabber/ACT_LED_1 -> VDD
- U7 pad 12: /Grabber/ACT_LED_2 -> unconnected-(U7-PH0-Pad12)
- U7 pad 13: /Grabber/CAM_HREF -> unconnected-(U7-PH1-Pad13)
- U7 pad 14: /Grabber/CAM_PWDN -> unconnected-(U7-NRST-Pad14)
- U7 pad 15: /Grabber/CAM_RESET -> unconnected-(U7-PC0-Pad15)
- U7 pad 19: /Grabber/CAM_D0 -> VDD
- U7 pad 20: /Grabber/CAM_D1 -> GND
- U7 pad 21: /Grabber/CAM_D2 -> VDD
- U7 pad 22: /Grabber/CAM_D3 -> VDD
- U7 pad 23: /Grabber/CAM_D4 -> /Grabber/ACT_LED_1
- U7 pad 24: /Grabber/CAM_D5 -> /Grabber/ACT_LED_2
- U7 pad 25: /Grabber/CAM_D6 -> /Grabber/CAM_PWDN
- U7 pad 26: /Grabber/CAM_D7 -> /Grabber/CAM_RESET
- U7 pad 27: /Grabber/CAM_PCLK -> GND
- U7 pad 28: /Grabber/CAM_XCLK -> VDD
- U7 pad 29: /Grabber/CAM_VSYNC -> /Grabber/CAM_HREF
- U7 pad 3: unconnected-(U7-PC15-Pad3) -> /Grabber/CAM_D4
- U7 pad 31: unconnected-(U7-PC7-Pad31) -> /Grabber/CAM_PCLK
- U7 pad 33: /Grabber/SCL -> unconnected-(U7-PC4-Pad33)
- U7 pad 34: /Grabber/SDA -> unconnected-(U7-PC5-Pad34)
- U7 pad 35: /Grabber/SWDIO -> unconnected-(U7-PB0-Pad35)
- U7 pad 36: /Grabber/SWCLK -> unconnected-(U7-PB1-Pad36)
- U7 pad 4: VDD -> unconnected-(U7-PE5-Pad4)
- U7 pad 46: /SPI_DI -> unconnected-(U7-PE15-Pad46)
- U7 pad 47: /SPI_CK -> /Grabber/SCL
- U7 pad 48: /SPI_CS -> /Grabber/SDA
- U7 pad 5: VDD -> unconnected-(U7-PE6-Pad5)
- U7 pad 7: GND -> unconnected-(U7-PC13-Pad7)
Routing:
- net VDD: track 133.9 -> 415.2 mm, vias 6 -> 9
- net +5V-A: track 109.0 -> 347.3 mm, vias 65 -> 272
- net /SPI_CS: track 50.0 -> 259.3 mm, vias 2 -> 4
- net /SPI_DI: track 52.1 -> 257.6 mm, vias 2 -> 4
- net /SPI_CK: track 52.3 -> 257.6 mm, vias 2 -> 4
- net LS24: track 32.0 -> 203.6 mm
- net LS31: track 38.0 -> 208.2 mm
- net LS29: track 36.3 -> 206.5 mm
- net LS27: track 34.5 -> 204.8 mm
- net LS28: track 35.4 -> 205.7 mm
- net LS30: track 37.1 -> 207.4 mm
- net LS26: track 33.7 -> 204.0 mm
- net LS25: track 32.8 -> 202.6 mm
- net LS7: track 70.4 -> 204.6 mm
- net LS6: track 71.2 -> 205.4 mm
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Other:
- board size 155.1 x 39.1 mm -> 556 x 39.1 mm

Commit message: Is this perfectionism…? (Submit for fab)
Parts:
- moved G*** 62.5 mm to (-140.8, 48.6)
Routing:
- net VDD: track 415.2 -> 409.5 mm, vias 9 -> 10
- net /Grabber/CAM_PCLK: track 36.7 -> 35.1 mm
- net /Grabber/CAM_HREF: track 43.1 -> 44.1 mm
- net /Grabber/CAM_D4: track 43.4 -> 44.3 mm
- net /SPI_CS: track 259.3 -> 258.7 mm
- net /SPI_DI: track 257.6 -> 257.1 mm, vias 4 -> 2
- net /Grabber/CAM_D7: track 39.6 -> 39.1 mm
Other:
- board text added: "24-SmEst"
- board text added: "Rev. 2"
- board text removed: "24-Soak"
- board text removed: "Rev. 1"

Commit message: Revise board routing
Parts:
- moved G*** 0.25 mm to (-141.1, 48.6)
Routing:
- net /Grabber/CAM_PCLK: track 35.1 -> 36.4 mm
- net VDD: track 409.5 -> 408.9 mm
- net /Grabber/CAM_D6: track 39.7 -> 39.1 mm
- net /Grabber/SCL: track 47.3 -> 47.4 mm, vias 0 -> 1
Other:
- outline, holes or cut-outs redrawn
