File: Distributor/hw/Distributor.kicad_pcb (KiCad board)
At the start: 2 copper layers, 556 x 39.1 mm, 95 parts, among them J1 Conn_01x04, J100 Conn_01x03, J101 Conn_01x03, J102 Conn_01x03, J103 Conn_01x03, J104 Conn_01x03, J105 Conn_01x03, J106 Conn_01x03, J107 Conn_01x03, J108 Conn_01x03, J109 Conn_01x03, J110 Conn_01x03, J111 Conn_01x03, J112 Conn_01x03, J113 Conn_01x03, J114 Conn_01x03, J115 Conn_01x03, J116 Conn_01x03, J117 Conn_01x03, J118 Conn_01x03, J119 Conn_01x03, J120 Conn_01x03, J121 Conn_01x03, J122 Conn_01x03, J123 Conn_01x03, J124 Conn_01x03, J125 Conn_01x03, J126 Conn_01x03, J127 Conn_01x03, J128 Conn_01x03, J129 Conn_01x03, J130 Conn_01x03, J131 Conn_01x03, J2 Conn_01x06_MountingPin, J3 Conn_01x02, J4 Conn_01x02, J5 Conn_01x02, J6 Conn_01x02, J7 Conn_01x04, J8 Conn_01x06_MountingPin, J9 Conn_02x09_Odd_Even, U1 SPX3819M5-L-3-3, U2 STM32G030C8Tx, U3 SN74AHCT245PWR, U4 SN74AHCT245PWR, U5 SN74AHCT245PWR, U6 SN74AHCT245PWR, U7 STM32F407VETx, U8 MLX90640ESF-BAB-000-TU

Commit message: Fix wrong value of capacitors on VCAP pins
Parts:
- C21, C22: value 100n -> 2.2u
Changed lines of the file:
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@@
         (effects (font (size 1 1) (thickness 0.15)))
     )
-    (fp_text value "100n" (at 0 1.43 90) (layer "F.Fab")
+    (fp_text value "2.2u" (at 0 1.43 90) (layer "F.Fab")
         (effects (font (size 1 1) (thickness 0.15)))
     )
@@
         (effects (font (size 1 1) (thickness 0.15)))
     )
-    (fp_text value "100n" (at 0 1.43) (layer "F.Fab")
+    (fp_text value "2.2u" (at 0 1.43) (layer "F.Fab")
         (effects (font (size 1 1) (thickness 0.15)))
     )

Commit message: Update EDA document with actual values in assembly
Parts:
- C1: value 2.2u -> 4.7u
- D1, D7: value White -> Green
- D2, D8: value White -> Yellow
- D3, D4, D5, D6: value Green -> White
- R2, R8: value 4.7k TBD -> 10k
- R3, R9: value 4.7k TBD -> 7.5k
- R4, R5, R6, R7: value 6.8k TBD -> 10k
Changed lines of the file:
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@@
         (effects (font (size 1 1) (thickness 0.15)))
     )
-    (fp_text value "Green" (at 0 1.43 90) (layer "F.Fab")
+    (fp_text value "White" (at 0 1.43 90) (layer "F.Fab")
         (effects (font (size 1 1) (thickness 0.15)))
     )
@@
         (effects (font (size 1 1) (thickness 0.15)))
     )
-    (fp_text value "4.7k TBD" (at 0 1.43 90) (layer "F.Fab")
+    (fp_text value "10k" (at 0 1.43 90) (layer "F.Fab")
         (effects (font (size 1 1) (thickness 0.15)))
     )
@@
         (effects (font (size 1 1) (thickness 0.15)))
     )
-    (fp_text value "4.7k TBD" (at 0 1.43 90) (layer "F.Fab")
+    (fp_text value "7.5k" (at 0 1.43 90) (layer "F.Fab")
         (effects (font (size 1 1) (thickness 0.15)))
     )
@@
         (effects (font (size 1 1) (thickness 0.15)))
     )
-    (fp_text value "White" (at 0 1.43 90) (layer "F.Fab")
+    (fp_text value "Yellow" (at 0 1.43 90) (layer "F.Fab")
         (effects (font (size 1 1) (thickness 0.15)))
     )
@@
         (effects (font (size 1 1) (thickness 0.15)))
     )
-    (fp_text value "6.8k TBD" (at 0 1.43 90) (layer "F.Fab")
+    (fp_text value "10k" (at 0 1.43 90) (layer "F.Fab")
         (effects (font (size 1 1) (thickness 0.15)))
     )
@@
         (effects (font (size 1 1) (thickness 0.15)))
     )
-    (fp_text value "6.8k TBD" (at 0 1.43 90) (layer "F.Fab")
+    (fp_text value "10k" (at 0 1.43 90) (layer "F.Fab")
         (effects (font (size 1 1) (thickness 0.15)))
     )
@@
         (effects (font (size 1 1) (thickness 0.15)))
     )
-    (fp_text value "6.8k TBD" (at 0 1.43 90) (layer "F.Fab")
+    (fp_text value "10k" (at 0 1.43 90) (layer "F.Fab")
         (effects (font (size 1 1) (thickness 0.15)))
     )
@@
         (effects (font (size 1 1) (thickness 0.15)))
     )
-    (fp_text value "4.7k TBD" (at 0 1.43) (layer "F.Fab")
+    (fp_text value "10k" (at 0 1.43) (layer "F.Fab")
         (effects (font (size 1 1) (thickness 0.15)))
     )
@@
         (effects (font (size 1 1) (thickness 0.15)))
     )
-    (fp_text value "White" (at 0 1.43) (layer "F.Fab")
+    (fp_text value "Green" (at 0 1.43) (layer "F.Fab")
         (effects (font (size 1 1) (thickness 0.15)))
     )
@@
         (effects (font (size 1 1) (thickness 0.15)))
     )
-    (fp_text value "4.7k TBD" (at 0 1.43) (layer "F.Fab")
+    (fp_text value "7.5k" (at 0 1.43) (layer "F.Fab")
         (effects (font (size 1 1) (thickness 0.15)))
     )
@@
         (effects (font (size 1 1) (thickness 0.15)))
     )
-    (fp_text value "White" (at 0 1.43) (layer "F.Fab")
+    (fp_text value "Yellow" (at 0 1.43) (layer "F.Fab")
         (effects (font (size 1 1) (thickness 0.15)))
     )
@@
         (effects (font (size 1 1) (thickness 0.15)))
     )
-    (fp_text value "2.2u" (at 0 1.43) (layer "F.Fab")
+    (fp_text value "4.7u" (at 0 1.43) (layer "F.Fab")
         (effects (font (size 1 1) (thickness 0.15)))
     )
@@
         (effects (font (size 1 1) (thickness 0.15)))
     )
-    (fp_text value "Green" (at 0 1.43 90) (layer "F.Fab")
+    (fp_text value "White" (at 0 1.43 90) (layer "F.Fab")
         (effects (font (size 1 1) (thickness 0.15)))
     )
@@
         (effects (font (size 1 1) (thickness 0.15)))
     )
-    (fp_text value "6.8k TBD" (at 0 1.43 90) (layer "F.Fab")
+    (fp_text value "10k" (at 0 1.43 90) (layer "F.Fab")
         (effects (font (size 1 1) (thickness 0.15)))
     )
@@
         (effects (font (size 1 1) (thickness 0.15)))
     )
-    (fp_text value "Green" (at 0 1.43 90) (layer "F.Fab")
+    (fp_text value "White" (at 0 1.43 90) (layer "F.Fab")
         (effects (font (size 1 1) (thickness 0.15)))
     )
@@
         (effects (font (size 1 1) (thickness 0.15)))
     )
-    (fp_text value "White" (at 0 1.43 90) (layer "F.Fab")
+    (fp_text value "Green" (at 0 1.43 90) (layer "F.Fab")
         (effects (font (size 1 1) (thickness 0.15)))
     )
@@
         (effects (font (size 1 1) (thickness 0.15)))
     )
-    (fp_text value "Green" (at 0 1.43 90) (layer "F.Fab")
+    (fp_text value "White" (at 0 1.43 90) (layer "F.Fab")
         (effects (font (size 1 1) (thickness 0.15)))
     )
